Commit message: Add FK workspace visualization for new URDF, fix mesh paths, add old vs new comparison
Agent-Logs-Url: https://github.com/Sheepyyt/dual_arm_strawberry_planning/sessions/7dfc27e7-1c88-460d-a47e-639dbae95828

Co-authored-by: Sheepyyt <148667544+Sheepyyt@users.noreply.github.com>

File: urdf/berrybolter_arm.urdf (robot description, URDF)
Before this commit: robot berrybolter_arm, 11 links, 10 joints
Links:
- link base_link: geometry collision mesh filename=meshes_single_arm/collision/base_link.STL; visual mesh filename=meshes_single_arm/visual/base_link.STL
- link camera_link: geometry collision mesh filename=meshes_single_arm/collision/camera_link.STL; visual mesh filename=meshes_single_arm/visual/camera_link.STL
- link ee_link: geometry collision mesh filename=meshes_single_arm/collision/ee_link.STL; visual mesh filename=meshes_single_arm/visual/ee_link.STL
- link link1: geometry collision mesh filename=meshes_single_arm/collision/link1.STL; visual mesh filename=meshes_single_arm/visual/link1.STL
- link link2: geometry collision mesh filename=meshes_single_arm/collision/link2.STL; visual mesh filename=meshes_single_arm/visual/link2.STL
- link link3: geometry collision mesh filename=meshes_single_arm/collision/link3.STL; visual mesh filename=meshes_single_arm/visual/link3.STL
- link link4: geometry collision mesh filename=meshes_single_arm/collision/link4.STL; visual mesh filename=meshes_single_arm/visual/link4.STL
- link link5: geometry collision mesh filename=meshes_single_arm/collision/link5.STL; visual mesh filename=meshes_single_arm/visual/link5.STL
- link link6: geometry collision mesh filename=meshes_single_arm/collision/link6.STL; visual mesh filename=meshes_single_arm/visual/link6.STL
- link link7: geometry collision mesh filename=meshes_single_arm/collision/link7.STL; visual mesh filename=meshes_single_arm/visual/link7.STL

File: urdf/berrybolter_arm.urdf.xacro (robot description, xacro)
@@ -34,5 +34,5 @@
       <origin xyz="0 0 0" rpy="0 0 0" />
       <geometry>
-        <mesh filename="package://berrybolter_arm_description/meshes_single_arm/visual/base_link.STL" />
+        <mesh filename="meshes_single_arm/visual/base_link.STL" />
       </geometry>
       <material name="graphite_grey"/>
@@ -41,5 +41,5 @@
       <origin xyz="0 0 0" rpy="0 0 0" />
       <geometry>
-        <mesh filename="package://berrybolter_arm_description/meshes_single_arm/collision/base_link.STL" />
+        <mesh filename="meshes_single_arm/collision/base_link.STL" />
       </geometry>
     </collision>
@@ -54,12 +54,12 @@
       <origin xyz="0 0 0" rpy="0 0 0" />
       <geometry>
-        <mesh filename="package://berrybolter_arm_description/meshes_single_arm/visual/link1.STL" />
-      </geometry>
-      <material name="white_matte"/>
-    </visual>
-    <collision>
-      <origin xyz="0 0 0" rpy="0 0 0" />
-      <geometry>
-        <mesh filename="package://berrybolter_arm_description/meshes_single_arm/collision/link1.STL" />
+        <mesh filename="meshes_single_arm/visual/link1.STL" />
+      </geometry>
+      <material name="white_matte"/>
+    </visual>
+    <collision>
+      <origin xyz="0 0 0" rpy="0 0 0" />
+      <geometry>
+        <mesh filename="meshes_single_arm/collision/link1.STL" />
       </geometry>
     </collision>
@@ -81,12 +81,12 @@
       <origin xyz="0 0 0" rpy="0 0 0" />
       <geometry>
-        <mesh filename="package://berrybolter_arm_description/meshes_single_arm/visual/link2.STL" />
-      </geometry>
-      <material name="white_matte"/>
-    </visual>
-    <collision>
-      <origin xyz="0 0 0" rpy="0 0 0" />
-      <geometry>
-        <mesh filename="package://berrybolter_arm_description/meshes_single_arm/collision/link2.STL" />
+        <mesh filename="meshes_single_arm/visual/link2.STL" />
+      </geometry>
+      <material name="white_matte"/>
+    </visual>
+    <collision>
+      <origin xyz="0 0 0" rpy="0 0 0" />
+      <geometry>
+        <mesh filename="meshes_single_arm/collision/link2.STL" />
       </geometry>
     </collision>
@@ -108,12 +108,12 @@
       <origin xyz="0 0 0" rpy="0 0 0" />
       <geometry>
-        <mesh filename="package://berrybolter_arm_description/meshes_single_arm/visual/link3.STL" />
-      </geometry>
-      <material name="white_matte"/>
-    </visual>
-    <collision>
-      <origin xyz="0 0 0" rpy="0 0 0" />
-      <geometry>
-        <mesh filename="package://berrybolter_arm_description/meshes_single_arm/collision/link3.STL" />
+        <mesh filename="meshes_single_arm/visual/link3.STL" />
+      </geometry>
+      <material name="white_matte"/>
+    </visual>
+    <collision>
+      <origin xyz="0 0 0" rpy="0 0 0" />
+      <geometry>
+        <mesh filename="meshes_single_arm/collision/link3.STL" />
       </geometry>
     </collision>
@@ -135,12 +135,12 @@
       <origin xyz="0 0 0" rpy="0 0 0" />
       <geometry>
-        <mesh filename="package://berrybolter_arm_description/meshes_single_arm/visual/link4.STL" />
-      </geometry>
-      <material name="white_matte"/>
-    </visual>
-    <collision>
-      <origin xyz="0 0 0" rpy="0 0 0" />
-      <geometry>
-        <mesh filename="package://berrybolter_arm_description/meshes_single_arm/collision/link4.STL" />
+        <mesh filename="meshes_single_arm/visual/link4.STL" />
+      </geometry>
+      <material name="white_matte"/>
+    </visual>
+    <collision>
+      <origin xyz="0 0 0" rpy="0 0 0" />
+      <geometry>
+        <mesh filename="meshes_single_arm/collision/link4.STL" />
       </geometry>
     </collision>
@@ -162,12 +162,12 @@
       <origin xyz="0 0 0" rpy="0 0 0" />
       <geometry>
-        <mesh filename="package://berrybolter_arm_description/meshes_single_arm/visual/link5.STL" />
-      </geometry>
-      <material name="white_matte"/>
-    </visual>
-    <collision>
-      <origin xyz="0 0 0" rpy="0 0 0" />
-      <geometry>
-        <mesh filename="package://berrybolter_arm_description/meshes_single_arm/collision/link5.STL" />
+        <mesh filename="meshes_single_arm/visual/link5.STL" />
+      </geometry>
+      <material name="white_matte"/>
+    </visual>
+    <collision>
+      <origin xyz="0 0 0" rpy="0 0 0" />
+      <geometry>
+        <mesh filename="meshes_single_arm/collision/link5.STL" />
       </geometry>
     </collision>
@@ -189,12 +189,12 @@
       <origin xyz="0 0 0" rpy="0 0 0" />
       <geometry>
-        <mesh filename="package://berrybolter_arm_description/meshes_single_arm/visual/link6.STL" />
-      </geometry>
-      <material name="white_matte"/>
-    </visual>
-    <collision>
-      <origin xyz="0 0 0" rpy="0 0 0" />
-      <geometry>
-        <mesh filename="package://berrybolter_arm_description/meshes_single_arm/collision/link6.STL" />
+        <mesh filename="meshes_single_arm/visual/link6.STL" />
+      </geometry>
+      <material name="white_matte"/>
+    </visual>
+    <collision>
+      <origin xyz="0 0 0" rpy="0 0 0" />
+      <geometry>
+        <mesh filename="meshes_single_arm/collision/link6.STL" />
       </geometry>
     </collision>
@@ -216,5 +216,5 @@
       <origin xyz="0 0 0" rpy="0 0 0" />
       <geometry>
-        <mesh filename="package://berrybolter_arm_description/meshes_single_arm/visual/link7.STL" />
+        <mesh filename="meshes_single_arm/visual/link7.STL" />
       </geometry>
       <material name="silver_metallic"/>
@@ -223,5 +223,5 @@
       <origin xyz="0 0 0" rpy="0 0 0" />
       <geometry>
-        <mesh filename="package://berrybolter_arm_description/meshes_single_arm/collision/link7.STL" />
+        <mesh filename="meshes_single_arm/collision/link7.STL" />
       </geometry>
     </collision>
@@ -243,5 +243,5 @@
       <origin xyz="0 0 0" rpy="0 0 0" />
       <geometry>
-        <mesh filename="package://berrybolter_arm_description/meshes_single_arm/visual/ee_link.STL" />
+        <mesh filename="meshes_single_arm/visual/ee_link.STL" />
       </geometry>
       <material name="graphite_grey"/>
@@ -250,5 +250,5 @@
       <origin xyz="0 0 0" rpy="0 0 0" />
       <geometry>
-        <mesh filename="package://berrybolter_arm_description/meshes_single_arm/collision/ee_link.STL" />
+        <mesh filename="meshes_single_arm/collision/ee_link.STL" />
       </geometry>
     </collision>
@@ -270,5 +270,5 @@
       <origin xyz="0 0 0" rpy="0 0 0" />
       <geometry>
-        <mesh filename="package://berrybolter_arm_description/meshes_single_arm/visual/camera_link.STL" />
+        <mesh filename="meshes_single_arm/visual/camera_link.STL" />
       </geometry>
       <material name="camera_black"/>
@@ -277,5 +277,5 @@
       <origin xyz="0 0 0" rpy="0 0 0" />
       <geometry>
-        <mesh filename="package://berrybolter_arm_description/meshes_single_arm/collision/camera_link.STL" />
+        <mesh filename="meshes_single_arm/collision/camera_link.STL" />
       </geometry>
     </collision>
