Commit message: Modified the urdf file.

File: urdf/dual_arm_ik_xy_centered.urdf (robot description, URDF)
Before this commit: robot berrybolter_dual_arm_minimal, 19 links, 18 joints
Joints:
- joint vehicle_to_left_arm: origin xyz=0.28336 0.22875 0.27926 rpy=0 0 -3.141592653589793 -> xyz=-0.28336 -0.22875 0.3126 rpy=0 0 0
- joint vehicle_to_right_arm: origin xyz=-0.28336 -0.22875 0.3126 rpy=0 0 0 -> xyz=0.28336 0.22875 0.27926 rpy=0 0 -3.141592653589793

Commit message: Updated the URDF file.

File: urdf/dual_arm_ik_xy_centered.urdf (robot description, URDF)
Before this commit: robot berrybolter_dual_arm_minimal, 19 links, 18 joints
Joints:
- joint left_arm_ee_joint: origin xyz=5.31363646517069E-05 -0.000500000000002027 0.0665000000000101 rpy=0 0 0 -> xyz=5.3136E-05 -0.0005 0.0665 rpy=0 0 0
- joint left_arm_joint1: limit lower=0.01 upper=0.2 effort=0 velocity=0 -> lower=0.001 upper=0.235 effort=0 velocity=0
- joint left_arm_joint3: limit lower=0.01 upper=0.45 effort=100 velocity=100 -> lower=0.001 upper=0.45 effort=100 velocity=100
- joint left_arm_joint4: limit lower=-3.14 upper=-0.01 effort=100 velocity=100 -> lower=-3.25 upper=-0.001 effort=100 velocity=100; origin xyz=0.044 -0.0011758 -0.043462 rpy=-3.141592653589793 0 1.666 -> xyz=0.044 -0.0011758 -0.044462 rpy=-3.1416 0 1.666
- joint left_arm_joint5: limit lower=-4.8 upper=-0.01 effort=100 velocity=100 -> lower=-3.6 upper=-0.001 effort=100 velocity=100; origin xyz=0.17 0 0.013 rpy=-3.141592653589793 0 2.3966 -> xyz=0.12 0 0.011 rpy=-3.1416 0 2.3966
- joint left_arm_joint6: axis 0 0 1 -> 0 0 -1; limit lower=-3.869 upper=-0.01 effort=100 velocity=100 -> lower=0 upper=4.0 effort=100 velocity=100; origin xyz=0.15961 0.00055813 -0.031456 rpy=0 0 1.9687 -> xyz=0.10972 0.069719 -0.048 rpy=0 0 1.9745
- joint left_arm_joint7: origin xyz=0.074633 -0.00014535 -0.038644 rpy=-1.570796326794897 0 -1.570796326794897 -> xyz=0.050498 0.034219 -0.02501 rpy=-1.5708 0 -0.97525
- joint right_arm_ee_joint: origin xyz=5.31363646517069E-05 -0.000500000000002027 0.0665000000000101 rpy=0 0 0 -> xyz=5.3136E-05 -0.0005 0.0665 rpy=0 0 0
- joint right_arm_joint1: limit lower=0.01 upper=0.2 effort=0 velocity=0 -> lower=0.001 upper=0.235 effort=0 velocity=0
- joint right_arm_joint3: limit lower=0.01 upper=0.45 effort=100 velocity=100 -> lower=0.001 upper=0.45 effort=100 velocity=100
- joint right_arm_joint4: limit lower=-3.14 upper=-0.01 effort=100 velocity=100 -> lower=-3.25 upper=-0.001 effort=100 velocity=100; origin xyz=0.044 -0.0011758 -0.043462 rpy=-3.141592653589793 0 1.666 -> xyz=0.044 -0.0011758 -0.044462 rpy=-3.1416 0 1.666
- joint right_arm_joint5: limit lower=-4.8 upper=-0.01 effort=100 velocity=100 -> lower=-3.6 upper=-0.001 effort=100 velocity=100; origin xyz=0.17 0 0.013 rpy=-3.141592653589793 0 2.3966 -> xyz=0.12 0 0.011 rpy=-3.1416 0 2.3966
- joint right_arm_joint6: axis 0 0 1 -> 0 0 -1; limit lower=-3.869 upper=-0.01 effort=100 velocity=100 -> lower=0 upper=4.0 effort=100 velocity=100; origin xyz=0.15961 0.00055813 -0.031456 rpy=0 0 1.9687 -> xyz=0.10972 0.069719 -0.048 rpy=0 0 1.9745
- joint right_arm_joint7: origin xyz=0.074633 -0.00014535 -0.038644 rpy=-1.570796326794897 0 -1.570796326794897 -> xyz=0.050498 0.034219 -0.02501 rpy=-1.5708 0 -0.97525
